Commit message: camera,lidar urdf and launch files, gazebo + ros2 control choos between

File: src/robomealmate/description/robot.urdf.xacro (robot description, xacro)
@@ -1,7 +1,13 @@
 <?xml version="1.0"?>
 <robot xmlns:xacro="http://www.ros.org/wiki/xacro"  name="robot">
+<xacro:arg name="use_ros2_controller" default="true"/>
 <xacro:include filename="robot_core.xacro"/>
-<!--<xacro:include filename="gazebo_controller.xacro"/>-->
+<xacro:if value="$(arg use_ros2_controller)">
+    <xacro:include filename="ros2_controller.xacro"/>
+</xacro:if>
+<xacro:unless value="$(arg use_ros2_controller)">
+    <xacro:include filename="gazebo_controller.xacro"/>
+</xacro:unless>
 <xacro:include filename="lidar.xacro"/>
-<xacro:include filename="ros2_controller.xacro"/>
+ <xacro:include filename="camera.xacro"/>
 </robot>

File: src/robomealmate/description/robot_core.xacro (robot description, xacro)
@@ -182,5 +182,5 @@
     <collision>
       <geometry>
-        <box size="0.15 0.20 0.40"/>
+        <box size="0.15 0.45 0.40"/>
       </geometry>
     </collision>

File: src/robomealmate/description/ros2_controller.xacro (robot description, xacro)
@@ -48,5 +48,5 @@
         </joint>
     </ros2_control>
-    <!--<ros2_control name="GazeboSystem" type="system">
+    <!-- <ros2_control name="GazeboSystem" type="system">
         <hardware>
             <plugin>gazebo_ros2_control/GazeboSystem</plugin>
@@ -84,5 +84,5 @@
             <state_interface name="position"/>
         </joint>
-    </ros2_control>-->
+    </ros2_control> -->
     <gazebo>
         <plugin name="gazebo_ros2_control" filename="libgazebo_ros2_control.so">
