Commit message: synch with VM

File: src/robomealmate/description/lidar.xacro (robot description, xacro)
@@ -19,5 +19,5 @@
       </geometry>
     </collision>
-    <xacro:inertial_cylinder  mass="0.10" radius="0.05" length="0.04">
+    <xacro:inertial_cylinder  mass="0.01" radius="0.05" length="0.04">
       <origin xyz="0.0 0.0 0.0" rpy= "0.0 0.0 0.0"/>
     </xacro:inertial_cylinder>

File: src/robomealmate/description/robot.urdf.xacro (robot description, xacro)
@@ -10,4 +10,4 @@
 </xacro:unless>
 <xacro:include filename="lidar.xacro"/>
- <xacro:include filename="camera.xacro"/>
+<xacro:include filename="camera.xacro"/>
 </robot>

File: src/robomealmate/description/robot_core.xacro (robot description, xacro)
@@ -26,4 +26,11 @@
     </xacro:inertial_box>
   </link>
+  <link name="base_footprint">
+  </link>
+  <joint name="base_footprint_joint" type="fixed">
+    <parent link="base"/>
+    <child link="base_footprint"/>
+    <origin xyz="0 0 0.0" rpy="0 0 0"/>
+  </joint>
   <!--front left wheel-->
   <joint name="front_left_wheel_joint" type="continuous">

File: src/robomealmate/description/ros2_controller.xacro (robot description, xacro)
@@ -1,5 +1,5 @@
 <?xml version="1.0"?>
 <robot xmlns:xacro="http://www.ros.org/wiki/xacro" name="robot">
-    <ros2_control name="RealRobot" type="system">
+    <!-- <ros2_control name="RealRobot" type="system">
         <hardware>
             <plugin>diffdrive_arduino/DiffDriveArduino</plugin>
@@ -47,6 +47,6 @@
             <state_interface name="position"/>
         </joint>
-    </ros2_control>
-    <!-- <ros2_control name="GazeboSystem" type="system">
+    </ros2_control> -->
+    <ros2_control name="GazeboSystem" type="system">
         <hardware>
             <plugin>gazebo_ros2_control/GazeboSystem</plugin>
@@ -84,5 +84,5 @@
             <state_interface name="position"/>
         </joint>
-    </ros2_control> -->
+    </ros2_control>
     <gazebo>
         <plugin name="gazebo_ros2_control" filename="libgazebo_ros2_control.so">
