Commit message: rplidar driver, simulation control, modfications, slam config, joystick config, twist muxconfig, camera+lidar launch files, ready for nav2

File: src/robomealmate/description/gazebo_controller.xacro (robot description, xacro)
@@ -16,5 +16,5 @@
             <!-- Output -->
             <odometry_frame>odom</odometry_frame>
-            <robot_base_frame>base</robot_base_frame>
+            <robot_base_frame>base_link</robot_base_frame>
             <publish_odom>true</publish_odom>
             <publish_odom_tf>true</publish_odom_tf>

File: src/robomealmate/description/lidar.xacro (robot description, xacro)
@@ -3,5 +3,5 @@
     <xacro:include filename="inertial_macros.xacro"/>
   <joint name="laser_joint" type="fixed">
-    <parent link="base"/>
+    <parent link="base_link"/>
     <child link="laser_frame"/>
     <origin xyz="0.25 0.0 0.17" rpy="0 0 0"/>

File: src/robomealmate/description/robot.urdf.xacro (robot description, xacro)
@@ -2,4 +2,5 @@
 <robot xmlns:xacro="http://www.ros.org/wiki/xacro"  name="robot">
 <xacro:arg name="use_ros2_controller" default="true"/>
+<xacro:arg name="sim_mode" default="false"/>
 <xacro:include filename="robot_core.xacro"/>
 <xacro:if value="$(arg use_ros2_controller)">

File: src/robomealmate/description/robot_core.xacro (robot description, xacro)
@@ -8,5 +8,5 @@
     <color rgba="0 0 0 1"/>
   </material>
-  <link name="base">
+  <link name="base_link">
     <visual>
       <origin xyz="0.15 0.0 0.075"/>
@@ -29,5 +29,5 @@
   </link>
   <joint name="base_footprint_joint" type="fixed">
-    <parent link="base"/>
+    <parent link="base_link"/>
     <child link="base_footprint"/>
     <origin xyz="0 0 0.0" rpy="0 0 0"/>
@@ -35,5 +35,5 @@
   <!--front left wheel-->
   <joint name="front_left_wheel_joint" type="continuous">
-    <parent link="base"/>
+    <parent link="base_link"/>
     <child link="front_left_wheel"/>
     <origin xyz="0.25 0.32 0.0" rpy="-${pi/2} 0.0 0.0"/>
@@ -58,5 +58,5 @@
     <!--front right wheel-->
   <joint name="front_right_wheel_joint" type="continuous">
-    <parent link="base"/>
+    <parent link="base_link"/>
     <child link="front_right_wheel"/>
     <origin xyz="0.25 -0.32 0.0" rpy=" ${pi/2} 0.0 0.0"/>
@@ -81,5 +81,5 @@
   <!--back left wheel-->
   <joint name="back_left_wheel_joint" type="continuous">
-    <parent link="base"/>
+    <parent link="base_link"/>
     <child link="back_left_wheel"/>
     <origin xyz="0.05 0.32 0.0" rpy="-${pi/2} 0.0 0.0"/>
@@ -104,5 +104,5 @@
   <!--back right wheel-->
   <joint name="back_right_wheel_joint" type="continuous">
-    <parent link="base"/>
+    <parent link="base_link"/>
     <child link="back_right_wheel"/>
     <origin xyz="0.05 -0.32 0.0" rpy=" ${pi/2} 0.0 0.0"/>
@@ -127,5 +127,5 @@
   <!--Left Feet-->
   <joint name="left_feet_joint" type="fixed">
-    <parent link="base"/>
+    <parent link="base_link"/>
     <child link="left_feet"/>
     <origin xyz="0.15 0.15 0.34"/>
@@ -151,5 +151,5 @@
   <!--Right Feet-->
   <joint name="right_feet_joint" type="fixed">
-    <parent link="base"/>
+    <parent link="base_link"/>
     <child link="right_feet"/>
     <origin xyz="0.15 -0.15 0.34"/>
@@ -175,5 +175,5 @@
   <!-- Body -->
   <joint name="body_joint" type="fixed">
-    <parent link="base"/>
+    <parent link="base_link"/>
     <child link="body"/>
     <origin xyz="0.15 0.0 0.73"/>
@@ -198,5 +198,5 @@
   <!--head-->
   <joint name="head_joint" type="fixed">
-    <parent link="base"/>
+    <parent link="base_link"/>
     <child link="head"/>
     <origin xyz="0.15 0.0 1.08"/>
@@ -219,5 +219,5 @@
     </xacro:inertial_box>
   </link>
-  <gazebo reference="base">
+  <gazebo reference="base_link">
     <material>Gazebo/Blue</material>
   </gazebo>

File: src/robomealmate/description/ros2_controller.xacro (robot description, xacro)
@@ -1,92 +1,97 @@
 <?xml version="1.0"?>
 <robot xmlns:xacro="http://www.ros.org/wiki/xacro" name="robot">
-    <!-- <ros2_control name="RealRobot" type="system">
-        <hardware>
-            <plugin>diffdrive_arduino/DiffDriveArduino</plugin>
-            <param name="num_wheel_pairs">2</param>
-            <param name="front_left_wheel_name">front_left_wheel_joint</param>
-            <param name="back_left_wheel_name">back_left_wheel_joint</param>
-            <param name="front_right_wheel_name">front_right_wheel_joint</param>
-            <param name="back_right_wheel_name">back_right_wheel_joint</param>
-            <param name="loop_rate">30</param>
-            <param name="device_name">/dev/ttyACM0</param>
-            <param name="baud_rate">9600</param>
-            <param name="timeout">1000</param>
-            <param name="enc_counts_per_rev">1920</param>
-        </hardware>
-        <joint name="front_left_wheel_joint">
-            <command_interface name="velocity">
-                <param name="min">-10.0</param>
-                <param name="max">10.0</param>
-            </command_interface>
-            <state_interface name="velocity"/>
-            <state_interface name="position"/>
-        </joint>
-        <joint name="front_right_wheel_joint">
-            <command_interface name="velocity">
-                <param name="min">-10.0</param>
-                <param name="max">10.0</param>
-            </command_interface>
-            <state_interface name="velocity"/>
-            <state_interface name="position"/>
-        </joint>
-        <joint name="back_left_wheel_joint">
-            <command_interface name="velocity">
-                <param name="min">-10.0</param>
-                <param name="max">10.0</param>
-            </command_interface>
-            <state_interface name="velocity"/>
-            <state_interface name="position"/>
-        </joint>
-        <joint name="back_right_wheel_joint">
-            <command_interface name="velocity">
-                <param name="min">-10.0</param>
-                <param name="max">10.0</param>
-            </command_interface>
-            <state_interface name="velocity"/>
-            <state_interface name="position"/>
-        </joint>
-    </ros2_control> -->
-    <ros2_control name="GazeboSystem" type="system">
-        <hardware>
-            <plugin>gazebo_ros2_control/GazeboSystem</plugin>
-        </hardware>
-        <joint name="front_left_wheel_joint">
-            <command_interface name="velocity">
-                <param name="min">-10.0</param>
-                <param name="max">10.0</param>
-            </command_interface>
-            <state_interface name="velocity"/>
-            <state_interface name="position"/>
-        </joint>
-        <joint name="front_right_wheel_joint">
-            <command_interface name="velocity">
-                <param name="min">-10.0</param>
-                <param name="max">10.0</param>
-            </command_interface>
-            <state_interface name="velocity"/>
-            <state_interface name="position"/>
-        </joint>
-        <joint name="back_left_wheel_joint">
-            <command_interface name="velocity">
-                <param name="min">-10.0</param>
-                <param name="max">10.0</param>
-            </command_interface>
-            <state_interface name="velocity"/>
-            <state_interface name="position"/>
-        </joint>
-        <joint name="back_right_wheel_joint">
-            <command_interface name="velocity">
-                <param name="min">-10.0</param>
-                <param name="max">10.0</param>
-            </command_interface>
-            <state_interface name="velocity"/>
-            <state_interface name="position"/>
-        </joint>
-    </ros2_control>
-    <gazebo>
-        <plugin name="gazebo_ros2_control" filename="libgazebo_ros2_control.so">
-            <parameters>$(find robomealmate)/config/controller.yaml</parameters>
-        </plugin>
-    </gazebo>
+    <xacro:if value="$(arg sim_mode)">
+        <ros2_control name="GazeboSystem" type="system">
+            <hardware>
+                <plugin>gazebo_ros2_control/GazeboSystem</plugin>
+            </hardware>
+            <joint name="front_left_wheel_joint">
+                <command_interface name="velocity">
+                    <param name="min">-10.0</param>
+                    <param name="max">10.0</param>
+                </command_interface>
+                <state_interface name="velocity"/>
+                <state_interface name="position"/>
+            </joint>
+            <joint name="front_right_wheel_joint">
+                <command_interface name="velocity">
+                    <param name="min">-10.0</param>
+                    <param name="max">10.0</param>
+                </command_interface>
+                <state_interface name="velocity"/>
+                <state_interface name="position"/>
+            </joint>
+            <joint name="back_left_wheel_joint">
+                <command_interface name="velocity">
+                    <param name="min">-10.0</param>
+                    <param name="max">10.0</param>
+                </command_interface>
+                <state_interface name="velocity"/>
+                <state_interface name="position"/>
+            </joint>
+            <joint name="back_right_wheel_joint">
+                <command_interface name="velocity">
+                    <param name="min">-10.0</param>
+                    <param name="max">10.0</param>
+                </command_interface>
+                <state_interface name="velocity"/>
+                <state_interface name="position"/>
+            </joint>
+        </ros2_control>
+        <gazebo>
+            <plugin name="gazebo_ros2_control" filename="libgazebo_ros2_control.so">
+                <parameters>$(find robomealmate)/config/controller.yaml</parameters>
+                <parameters>$(find robomealmate)/config/sim_mode_controller.yaml</parameters>
+            </plugin>
+        </gazebo>
+    </xacro:if>
+    <xacro:unless value="$(arg sim_mode)">
+        <ros2_control name="RealRobot" type="system">
+            <hardware>
+                <plugin>diffdrive_arduino/DiffDriveArduino</plugin>
+                <param name="num_wheel_pairs">2</param>
+                <param name="front_left_wheel_name">front_left_wheel_joint</param>
+                <param name="back_left_wheel_name">back_left_wheel_joint</param>
+                <param name="front_right_wheel_name">front_right_wheel_joint</param>
+                <param name="back_right_wheel_name">back_right_wheel_joint</param>
+                <param name="loop_rate">30</param>
+                <param name="device_name">/dev/ttyACM0</param>
+                <param name="baud_rate">9600</param>
+                <param name="timeout">1000</param>
+                <param name="enc_counts_per_rev">1920</param>
+            </hardware>
+            <joint name="front_left_wheel_joint">
+                <command_interface name="velocity">
+                    <param name="min">-10.0</param>
+                    <param name="max">10.0</param>
+                </command_interface>
+                <state_interface name="velocity"/>
+                <state_interface name="position"/>
+            </joint>
+            <joint name="front_right_wheel_joint">
+                <command_interface name="velocity">
+                    <param name="min">-10.0</param>
+                    <param name="max">10.0</param>
+                </command_interface>
+                <state_interface name="velocity"/>
+                <state_interface name="position"/>
+            </joint>
+            <joint name="back_left_wheel_joint">
+                <command_interface name="velocity">
+                    <param name="min">-10.0</param>
+                    <param name="max">10.0</param>
+                </command_interface>
+                <state_interface name="velocity"/>
+                <state_interface name="position"/>
+            </joint>
+            <joint name="back_right_wheel_joint">
+                <command_interface name="velocity">
+                    <param name="min">-10.0</param>
+                    <param name="max">10.0</param>
+                </command_interface>
+                <state_interface name="velocity"/>
+                <state_interface name="position"/>
+            </joint>
+        </ros2_control>
+    </xacro:unless>
 </robot>
